File: Eagle PCB/layer1.brd (EAGLE design)
At the start: 196 x 185.3 mm, 227 parts, among them M1C1 33nF, M1C2 680uF, M1C3 1.0uF, M1D1 RED, M1D2 BLUE, M1J1 XT30PB-F, M1Q1 AOD482, M1R1 1k, M1R10 1k, M1R11 10k, M1R12 4.7k, M1R2 1k, M1R3 3.3k, M1R4 3.3k, M1R5 1k, M1R6 1k, M1R7 1k, M1R8 10k, M1R9 10k, M2C1 33nF, M2C2 680uF, M2C3 1.0uF, M2D1 RED, M2D2 BLUE, M2J1 XT30PB-F, M2Q1 AOD482, M2R1 1k, M2R10 1k, M2R11 10k, M2R12 4.7k, M2R2 1k, M2R3 3.3k, M2R4 3.3k, M2R5 1k, M2R6 1k, M2R7 1k, M2R8 10k, M2R9 10k, M3C1 33nF, M3C2 680uF, M3C3 1.0uF, M3D1 RED, M3D2 BLUE, M3J1 XT30PB-F, M3Q1 AOD482, M3R1 1k, M3R10 1k, M3R11 10k, M3R12 4.7k, M3R2 1k, M3R3 3.3k, M3R4 3.3k, M3R5 1k, M3R6 1k, M3R7 1k, M3R8 10k, M3R9 10k, M4C1 33nF, M4C2 680uF, M4C3 1.0uF, M4D1 RED, M4D2 BLUE, M4J1 XT30PB-F, M4Q1 AOD482, M4R1 1k, M4R10 1k, M4R11 10k, M4R12 4.7k, M4R2 1k, M4R3 3.3k, M4R4 3.3k, M4R5 1k, M4R6 1k, M4R7 1k, M4R8 10k, M4R9 10k, X2 SM06B-SRSS-TB, Y1 8MHz

Commit message: Retard
Routing:
- net BL_CS: track 97.6 -> 98.6 mm
Changed lines of the file:
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@@
 <element name="RST" library="MY-LIBRARY" library_urn="urn:adsk.eagle:library:11016882" package="MOMENTARY_SWITCH_4X3" package3d_urn="urn:adsk.eagle:package:11016890/3" value="MOMENTARY_SWITCH_4X3" x="84.5" y="22" smashed="yes" rot="R270">
 <attribute name="NAME" x="86.525" y="21.678" size="1.27" layer="25"/>
+<attribute name="VALUE" x="84.052" y="52.502" size="1.27" layer="27" rot="R270"/>
 </element>
 <element name="BOOT" library="MY-LIBRARY" library_urn="urn:adsk.eagle:library:11016882" package="MOMENTARY_SWITCH_4X3" package3d_urn="urn:adsk.eagle:package:11016890/3" value="MOMENTARY_SWITCH_4X3" x="79.5" y="22" smashed="yes" rot="R270">
@@
 <wire x1="-5.21315" y1="48.75" x2="-8.881575" y2="45.081575" width="0.254" layer="16"/>
 <wire x1="76.8862" y1="-20.5138" x2="81" y2="-16.4" width="1.016" layer="1"/>
-<wire x1="50.0524125" y1="-37.9" x2="67.4386125" y2="-20.5138" width="1.016" layer="1"/>
-<wire x1="67.4386125" y1="-20.5138" x2="76.8862" y2="-20.5138" width="1.016" layer="1"/>
+<wire x1="55.7924125" y1="-37.9" x2="73.1786125" y2="-20.5138" width="1.016" layer="1"/>
+<wire x1="73.1786125" y1="-20.5138" x2="76.8862" y2="-20.5138" width="1.016" layer="1"/>
 <wire x1="33.5" y1="-31.65685" x2="32.893753125" y2="-32.263096875" width="0.504" layer="1"/>
 <wire x1="32.893753125" y1="-32.263096875" x2="31.8" y2="-33.35685" width="1.016" layer="1"/>
@@
 <wire x1="31.8" y1="-35.2" x2="32.81968125" y2="-36.21968125" width="1.016" layer="1"/>
 <wire x1="32.81968125" y1="-36.21968125" x2="36.28778125" y2="-36.21968125" width="1.016" layer="1"/>
-<wire x1="37.9681" y1="-37.9" x2="50.0524125" y2="-37.9" width="1.016" layer="1"/>
+<wire x1="37.9681" y1="-37.9" x2="55.7924125" y2="-37.9" width="1.016" layer="1"/>
 </signal>
 <signal name="GND">
@@
 <wire x1="15.73238125" y1="-28.68961875" x2="15.73238125" y2="-27.28604375" width="0.254" layer="1"/>
 <via x="22.9" y="4.3" extent="1-16" drill="0.508"/>
-<wire x1="18.056515625" y1="-17.1207375" x2="22.9" y2="-12.277253125" width="0.254" layer="1"/>
+<wire x1="20.676515625" y1="-14.5007375" x2="22.9" y2="-12.277253125" width="0.254" layer="1"/>
 <wire x1="22.9" y1="-12.277253125" x2="22.9" y2="4.3" width="0.254" layer="1"/>
-<wire x1="18.056515625" y1="-24.961909375" x2="18.056515625" y2="-17.1207375" width="0.254" layer="1"/>
+<wire x1="20.676515625" y1="-22.341909375" x2="20.676515625" y2="-14.5007375" width="0.254" layer="1"/>
 <wire x1="22.9" y1="4.3" x2="22.9" y2="8.3" width="0.254" layer="16"/>
 <wire x1="22.9" y1="8.3" x2="20.6" y2="10.6" width="0.254" layer="16"/>
@@
 <wire x1="20.6" y1="10.6" x2="21.127" y2="10.073" width="0.254" layer="1"/>
 <wire x1="21.127" y1="10.073" x2="21.127" y2="8" width="0.254" layer="1"/>
-<wire x1="15.73238125" y1="-27.28604375" x2="18.056515625" y2="-24.961909375" width="0.254" layer="1"/>
+<wire x1="15.73238125" y1="-27.28604375" x2="20.676515625" y2="-22.341909375" width="0.254" layer="1"/>
 <wire x1="18.8" y1="31.5" x2="18.12665625" y2="31.5" width="0.254" layer="1"/>
 <wire x1="18.12665625" y1="31.5" x2="17.8" y2="31.82665625" width="0.254" layer="1"/>
@@
 <wire x1="-20.789" y1="-7.5" x2="-17.9" y2="-10.389" width="0.254" layer="1"/>
 <wire x1="-17.9" y1="-10.389" x2="-17.9" y2="-17.1" width="0.254" layer="1"/>
-<wire x1="-17.9" y1="-17.1" x2="-16.289" y2="-18.711" width="0.254" layer="1"/>
+<wire x1="-17.9" y1="-17.1" x2="-15.789" y2="-19.211" width="0.254" layer="1"/>
 <via x="15.1" y="-19.1" extent="1-16" drill="0.508"/>
 <via x="31.2" y="-2.5" extent="1-16" drill="0.508"/>
@@
 <wire x1="29.6317625" y1="-2.511" x2="31.189" y2="-2.511" width="0.254" layer="16"/>
 <wire x1="-16.77861875" y1="17.73980625" x2="-20.789" y2="13.729425" width="0.254" layer="16"/>
-<wire x1="15.1" y1="-19.1" x2="14.711" y2="-18.711" width="0.254" layer="1"/>
-<wire x1="14.711" y1="-18.711" x2="-16.289" y2="-18.711" width="0.254" layer="1"/>
+<wire x1="14.989" y1="-19.211" x2="15.1" y2="-19.1" width="0.254" layer="1"/>
+<wire x1="14.989" y1="-19.211" x2="-15.789" y2="-19.211" width="0.254" layer="1"/>
 <wire x1="31.2" y1="-2.5" x2="41" y2="-2.5" width="0.254" layer="1"/>
 <wire x1="51.77" y1="-2.341" x2="46.3982375" y2="-2.341" width="0.254" layer="1"/>
@@
 <via x="-21.2" y="-25.5" extent="1-16" drill="0.508"/>
 <via x="3.6" y="42.4" extent="1-16" drill="0.508"/>
-<wire x1="-21.868628125" y1="-13.308628125" x2="-21.868628125" y2="8.474134375" width="0.254" layer="1"/>
+<wire x1="-23.088628125" y1="-12.088628125" x2="-23.088628125" y2="7.254134375" width="0.254" layer="1"/>
 <wire x1="-5.1888" y1="24.6539625" x2="-11.7397625" y2="18.103" width="0.254" layer="1"/>
 <wire x1="-21.2" y1="-25.5" x2="-21.2" y2="-15.297765625" width="0.254" layer="1"/>
 <wire x1="-21.2" y1="-15.297765625" x2="-20.676515625" y2="-14.77428125" width="0.254" layer="1"/>
 <wire x1="-20.676515625" y1="-14.77428125" x2="-20.676515625" y2="-14.500740625" width="0.254" layer="1"/>
-<wire x1="-20.676515625" y1="-14.500740625" x2="-21.868628125" y2="-13.308628125" width="0.254" layer="1"/>
+<wire x1="-20.676515625" y1="-14.500740625" x2="-23.088628125" y2="-12.088628125" width="0.254" layer="1"/>
 <wire x1="3.15" y1="42.85" x2="3.6" y2="42.4" width="0.254" layer="16"/>
 <wire x1="3.15" y1="44.758" x2="3.15" y2="42.85" width="0.254" layer="16"/>
@@
 <wire x1="-14.6" y1="17.011" x2="-14.4317625" y2="17.011" width="0.254" layer="1"/>
 <wire x1="-14.4317625" y1="17.011" x2="-13.3397625" y2="18.103" width="0.254" layer="1"/>
-<wire x1="-21.868628125" y1="8.474134375" x2="-14.6" y2="15.7427625" width="0.254" layer="1"/>
+<wire x1="-23.088628125" y1="7.254134375" x2="-14.6" y2="15.7427625" width="0.254" layer="1"/>
 <wire x1="-13.3397625" y1="18.103" x2="-11.7397625" y2="18.103" width="0.254" layer="1"/>
 <wire x1="2.6" y1="42.1" x2="2.5" y2="42" width="0.254" layer="1"/>
@@
 <wire x1="28.39895625" y1="-4.40104375" x2="26.9" y2="-5.9" width="0.254" layer="1"/>
 <via x="26.9" y="-5.9" extent="1-16" drill="0.508"/>
-<wire x1="26.9" y1="-5.9" x2="13.53" y2="-19.27" width="0.254" layer="16"/>
-<wire x1="13.53" y1="-19.27" x2="5.03" y2="-19.27" width="0.254" layer="16"/>
-<wire x1="5.03" y1="-19.27" x2="4.2" y2="-20.1" width="0.254" layer="16"/>
+<wire x1="26.9" y1="-5.9" x2="12.7" y2="-20.1" width="0.254" layer="16"/>
+<wire x1="12.7" y1="-20.1" x2="4.2" y2="-20.1" width="0.254" layer="16"/>
 <via x="4.2" y="-20.1" extent="1-16" drill="0.508"/>
-<wire x1="4.2" y1="-20.1" x2="1.16" y2="-20.1" width="0.254" layer="1"/>
-<wire x1="-0.4" y1="-21.7" x2="-0.4" y2="-21.66" width="0.254" layer="1"/>
-<wire x1="1.16" y1="-20.1" x2="-0.4" y2="-21.66" width="0.254" layer="1"/>
+<wire x1="4.2" y1="-20.1" x2="2.6" y2="-21.7" width="0.254" layer="1"/>
+<wire x1="2.6" y1="-21.7" x2="-0.4" y2="-21.7" width="0.254" layer="1"/>
 <via x="-0.4" y="-21.7" extent="1-16" drill="0.508"/>
 <via x="-17.9" y="-26.4" extent="1-16" drill="0.508"/>
@@
 <wire x1="-0.4" y1="-21.7" x2="-13.0427625" y2="-21.7" width="0.254" layer="16"/>
 <wire x1="-13.0427625" y1="-21.7" x2="-17.11038125" y2="-25.76761875" width="0.254" layer="16"/>
-<via x="-20.84" y="-9.41" extent="1-16" drill="0.508"/>
+<via x="-22" y="-8.5" extent="1-16" drill="0.508"/>
 <wire x1="-17.9" y1="-26.4" x2="-17.9" y2="-25.714475" width="0.254" layer="1"/>
-<wire x1="-19.108" y1="-11.142" x2="-20.84" y2="-9.41" width="0.254" layer="1"/>
+<wire x1="-19.108" y1="-11.392" x2="-22" y2="-8.5" width="0.254" layer="1"/>
 <wire x1="-17.9" y1="-25.714475" x2="-19.108" y2="-24.506475" width="0.254" layer="1"/>
-<wire x1="-19.108" y1="-24.506475" x2="-19.108" y2="-11.142" width="0.254" layer="1"/>
-<wire x1="-20.84" y1="-9.41" x2="-25.55" y2="-4.7" width="0.254" layer="16"/>
-<wire x1="-25.55" y1="-4.7" x2="-26.8" y2="-4.7" width="0.254" layer="16"/>
+<wire x1="-19.108" y1="-24.506475" x2="-19.108" y2="-11.392" width="0.254" layer="1"/>
+<wire x1="-22" y1="-8.5" x2="-25.8" y2="-4.7" width="0.254" layer="16"/>
+<wire x1="-25.8" y1="-4.7" x2="-26.8" y2="-4.7" width="0.254" layer="16"/>
 <via x="-26.8" y="-4.7" extent="1-16" drill="0.508"/>
 <wire x1="-26.8" y1="-4.7" x2="-27.7979125" y2="-4.7" width="0.254" layer="1"/>

Commit message: Fuck you
Parts:
- added V_BATT_M1, V_BATT_M2, V_BATT_M3, V_BATT_M4: 18AWG, JH:18AWG
Connections:
- net V_BATT: now also V_BATT_M1.P$1, V_BATT_M2.P$1, V_BATT_M3.P$1, V_BATT_M4.P$1
Changed lines of the file:
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@@
 <element name="RST" library="MY-LIBRARY" library_urn="urn:adsk.eagle:library:11016882" package="MOMENTARY_SWITCH_4X3" package3d_urn="urn:adsk.eagle:package:11016890/3" value="MOMENTARY_SWITCH_4X3" x="84.5" y="22" smashed="yes" rot="R270">
 <attribute name="NAME" x="86.525" y="21.678" size="1.27" layer="25"/>
-<attribute name="VALUE" x="84.052" y="52.502" size="1.27" layer="27" rot="R270"/>
 </element>
 <element name="BOOT" library="MY-LIBRARY" library_urn="urn:adsk.eagle:library:11016882" package="MOMENTARY_SWITCH_4X3" package3d_urn="urn:adsk.eagle:package:11016890/3" value="MOMENTARY_SWITCH_4X3" x="79.5" y="22" smashed="yes" rot="R270">
 <attribute name="NAME" x="72.825" y="21.478" size="1.27" layer="25"/>
-<attribute name="VALUE" x="78.248" y="33.498" size="1.27" layer="27" rot="R90"/>
 </element>
 <element name="U$15" library="MY-LIBRARY" library_urn="urn:adsk.eagle:library:11016882" package="2X7" package3d_urn="urn:adsk.eagle:package:16537177/2" value="CONN_07X2" x="91" y="6" smashed="yes" rot="R270">
@@
 <attribute name="NAME" x="-0.162" y="47.9" size="0.7112" layer="26" font="vector" ratio="18" rot="MR270" align="bottom-center"/>
 <attribute name="VALUE" x="1.362" y="47.9" size="0.7112" layer="28" font="vector" ratio="18" rot="MR270" align="top-center"/>
+</element>
+<element name="V_BATT_M1" library="JH" library_urn="urn:adsk.eagle:library:6027132" package="18AWG" package3d_urn="urn:adsk.eagle:package:16754415/1" value="18AWG" x="-113.2" y="-112.5" smashed="yes">
+<attribute name="NAME" x="-114.7" y="-111.2" size="0.6096" layer="25"/>
+</element>
+<element name="V_BATT_M2" library="JH" library_urn="urn:adsk.eagle:library:6027132" package="18AWG" package3d_urn="urn:adsk.eagle:package:16754415/1" value="18AWG" x="-113.2" y="-115.8" smashed="yes">
+<attribute name="NAME" x="-114.7" y="-114.5" size="0.6096" layer="25"/>
+</element>
+<element name="V_BATT_M3" library="JH" library_urn="urn:adsk.eagle:library:6027132" package="18AWG" package3d_urn="urn:adsk.eagle:package:16754415/1" value="18AWG" x="-113.2" y="-119.1" smashed="yes">
+<attribute name="NAME" x="-114.7" y="-117.8" size="0.6096" layer="25"/>
+</element>
+<element name="V_BATT_M4" library="JH" library_urn="urn:adsk.eagle:library:6027132" package="18AWG" package3d_urn="urn:adsk.eagle:package:16754415/1" value="18AWG" x="-113.2" y="-122.4" smashed="yes">
+<attribute name="NAME" x="-114.7" y="-121.1" size="0.6096" layer="25"/>
 </element>
 </elements>
@@
 <wire x1="32.81968125" y1="-36.21968125" x2="36.28778125" y2="-36.21968125" width="1.016" layer="1"/>
 <wire x1="37.9681" y1="-37.9" x2="55.7924125" y2="-37.9" width="1.016" layer="1"/>
+<contactref element="V_BATT_M1" pad="P$1"/>
+<contactref element="V_BATT_M4" pad="P$1"/>
+<contactref element="V_BATT_M2" pad="P$1"/>
+<contactref element="V_BATT_M3" pad="P$1"/>
+<wire x1="-113.2" y1="-119.1" x2="-113.2" y2="-122.4" width="0" layer="19" extent="1-1"/>
+<wire x1="-113.2" y1="-115.8" x2="-113.2" y2="-119.1" width="0" layer="19" extent="1-1"/>
+<wire x1="-113.2" y1="-112.5" x2="-113.2" y2="-115.8" width="0" layer="19" extent="1-1"/>
+<wire x1="-80.173" y1="-6.612" x2="-113.2" y2="-112.5" width="0" layer="19" extent="1-1"/>
 </signal>
 <signal name="GND">
