File: Eagle PCB/Layer 1.brd (EAGLE design)
At the start: 196 x 185.3 mm, 242 parts, among them M1C1 33nF, M1C2 680uF, M1C3 1.0uF, M1D1 RED, M1D2 BLUE, M1J1 XT30PB-F, M1Q1 AOD482, M1R1 1k, M1R10 1k, M1R11 10k, M1R12 4.7k, M1R2 1k, M1R3 3.3k, M1R4 3.3k, M1R5 1k, M1R6 1k, M1R7 1k, M1R8 10k, M1R9 10k, M2C1 33nF, M2C2 680uF, M2C3 1.0uF, M2D1 RED, M2D2 BLUE, M2J1 XT30PB-F, M2Q1 AOD482, M2R1 1k, M2R10 1k, M2R11 10k, M2R12 4.7k, M2R2 1k, M2R3 3.3k, M2R4 3.3k, M2R5 1k, M2R6 1k, M2R7 1k, M2R8 10k, M2R9 10k, M3C1 33nF, M3C2 680uF, M3C3 1.0uF, M3D1 RED, M3D2 BLUE, M3J1 XT30PB-F, M3Q1 AOD482, M3R1 1k, M3R10 1k, M3R11 10k, M3R12 4.7k, M3R2 1k, M3R3 3.3k, M3R4 3.3k, M3R5 1k, M3R6 1k, M3R7 1k, M3R8 10k, M3R9 10k, M4C1 33nF, M4C2 680uF, M4C3 1.0uF, M4D1 RED, M4D2 BLUE, M4J1 XT30PB-F, M4Q1 AOD482, M4R1 1k, M4R10 1k, M4R11 10k, M4R12 4.7k, M4R2 1k, M4R3 3.3k, M4R4 3.3k, M4R5 1k, M4R6 1k, M4R7 1k, M4R8 10k, M4R9 10k, X2 SM06B-SRSS-TB, Y1 8MHz

Commit message: Hello
Parts:
- removed 1C10: 22uF, JH:C1210
- removed 1C6: 4.7uF, JH:C0603
- removed 1C7: 220uF, SparkFun-Capacitors:EIA7343
- removed 1C8: 10nF, JH:C0603
- removed 1C9: 0.1uF, JH:C0603
- removed 1D2: SS54, JH:SMA-DIODE
- removed 1L2: 10uH, JH:SWPA8040
- removed 1R3: 10k, JH:R0603
- removed 1R4: 3.24k, JH:R0603
- removed BATT: XT30PB-F, JH:XT30PB-F
- removed GND_M1A, GND_M1B, GND_M3A, GND_M3B: 18AWG, JH:18AWG
- removed U2: (no value), JH:POWERPAD-SOIC-8
- added V_BATT_M1B, V_BATT_M2B, V_BATT_M3B, V_BATT_M4B: 18AWG, JH:18AWG
- moved GND_M4A 19.7 mm to (74.9, -4.50)
- moved S3 13.9 mm to (-28.2, -76.7), turned to 90 degrees
- moved X2 4.95 mm to (86.6, -16.5), turned to 270 degrees
- moved LDR 3.00 mm to (42.8, 74.0)
- moved LED 3.00 mm to (-41.2, 73.4)
- moved U$15 3.00 mm to (88.0, 6.00)
- moved 1L1 2.79 mm to (-84.3, 13.1)
- moved 1C2 2.79 mm to (-82.6, -3.91)
- moved 1C3 2.79 mm to (-79.9, 7.83)
- moved 1C5 2.79 mm to (-91.4, 1.39)
- moved 1R2 2.79 mm to (-85.3, -0.56)
- moved 1C1 2.79 mm to (-82.6, -1.52)
- moved U1 2.79 mm to (-82.0, 2.90)
- moved 1R1 2.79 mm to (-86.1, 7.72)
- moved LS1 2.79 mm to (-86.1, -7.60)
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- renumbered V_BATT_M1 to V_BATT_M1A, V_BATT_M2 to V_BATT_M2A, V_BATT_M3 to V_BATT_M3A, V_BATT_M4 to V_BATT_M4A
Connections:
- removed net 5V: 1C7.A, 1C9.1, 1L2.P2, 1R3.2
- removed net N$7: 1C8.2, 1D2.C, 1L2.P1, U2.8
- removed net N$8: 1R3.1, 1R4.2, U2.4
- removed net N$9: 1C8.1, U2.1
- net GND: now also M1C2.2, M1C3.2, M3C2.2, M3C3.2, M_BL.P18, M_BL.P19, M_BL.P20, M_BL.P26, M_BL.P27, M_BL.P28, M_FL.P18, M_FL.P19, M_FL.P20, M_FL.P26, M_FL.P27, M_FL.P28; no longer 1C10.2, 1C6.2, 1C7.C, 1C9.2, 1D2.A, 1R4.1, BATT.-, GND_M1B.P$1, GND_M3B.P$1, U2.6, U2.9, U2.P$1, U2.P$2, U2.P$3, U2.P$4, U2.P$5, U2.P$6
- net GND_M: no longer GND_M1A.P$1, GND_M3A.P$1, M1C2.2, M1C3.2, M3C2.2, M3C3.2, M_BL.P18, M_BL.P19, M_BL.P20, M_BL.P26, M_BL.P27, M_BL.P28, M_FL.P18, M_FL.P19, M_FL.P20, M_FL.P26, M_FL.P27, M_FL.P28
- net V_BATT: now also V_BATT_M1B.P$1, V_BATT_M2B.P$1, V_BATT_M3B.P$1, V_BATT_M4B.P$1; no longer 1C10.1, 1C6.1, BATT.+, U2.7
Routing:
- net V_BATT: track 412.5 -> 199.5 mm, vias 11 -> 5
- net GND_M: track 355.1 -> 150.3 mm, vias 27 -> 13
- net GND: track 373.5 -> 494.7 mm, vias 44 -> 63
- net BR_DIR: track 168.9 -> 141.3 mm
- net FR_OUTB: track 52.4 -> 31.2 mm, vias 2 -> 1
- net FL_OUTA: track 51.3 -> 32.7 mm
- net BL_OUTA: track 45.7 -> 28.4 mm
- net BL_OUTB: track 53.9 -> 37.0 mm
- net FR_OUTA: track 46.1 -> 30.1 mm, vias 1 -> 0
- net BR_OUTA: track 50.6 -> 34.7 mm
- net FL_OUTB: track 47.0 -> 34.6 mm
- net BR_OUTB: track 45.2 -> 33.0 mm, vias 3 -> 2
- net BR_PWM: track 112.0 -> 101.8 mm
- net 3.3V: track 595.3 -> 586.4 mm, vias 33 -> 32
- net FL_PWM: track 195.3 -> 186.7 mm, vias 9 -> 10
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- added copper zone on layer 1, net BL_OUTA
- added copper zone on layer 1, net BL_OUTB
- added copper zone on layer 1, net BR_OUTA
- added copper zone on layer 1, net BR_OUTB
- added copper zone on layer 1, net FL_OUTA
- added copper zone on layer 1, net FL_OUTB
- added copper zone on layer 1, net FR_OUTA
- added copper zone on layer 1, net RFR_OUTB
- added copper zone on layer 1, net V_BATT

Commit message: FUCK YOU
Parts:
- added 1C10: 22uF, JH:C1210
- added 1C6: 4.7uF, JH:C0603
- added 1C7: 220uF, SparkFun-Capacitors:EIA7343
- added 1C8: 10nF, JH:C0603
- added 1C9: 0.1uF, JH:C0603
- added 1D2: SS54, JH:SMA-DIODE
- added 1L2: 10uH, JH:SWPA8040
- added 1R3: 10k, JH:R0603
- added 1R4: 3.24k, JH:R0603
- added BATT: XT30PB-F, JH:XT30PB-F
- added U2: (no value), JH:POWERPAD-SOIC-8
Connections:
- new net 5V: 1C7.A, 1C9.1, 1L2.P2, 1R3.2
- new net N$3: 1C8.2, 1D2.C, 1L2.P1, U2.8
- new net N$5: 1R3.1, 1R4.2, U2.4
- new net N$6: 1C8.1, U2.1
- net GND: now also 1C10.2, 1C6.2, 1C7.C, 1C9.2, 1D2.A, 1R4.1, BATT.-, U2.6, U2.9, U2.P$1, U2.P$2, U2.P$3, U2.P$4, U2.P$5, U2.P$6
- net V_BATT: now also 1C10.1, 1C6.1, BATT.+, U2.7

Commit message: Hello
Parts:
- removed BATT: XT30PB-F, JH:XT30PB-F
- moved 1D2 107.5 mm to (-26.1, -72.4), turned to 180 degrees
- moved 1C6 104.1 mm to (-33.0, -57.9)
- moved 1L2 95.8 mm to (-26.8, -65.8), turned to 180 degrees
- moved 1C10 93.6 mm to (-31.3, -80.7)
- moved 1R3 89.9 mm to (-43.5, -80.7), turned to 180 degrees
- moved 1C9 89.6 mm to (-44.4, -84.0), turned to 270 degrees
- moved 1R4 89.2 mm to (-40.3, -81.5), turned to 90 degrees
- moved 1C8 88.0 mm to (-37.8, -72.4)
- moved 1C7 86.4 mm to (-44.4, -74.3), turned to 270 degrees
- moved U2 83.6 mm to (-37.8, -76.8)
- moved S3 4.70 mm to (-26.3, -81.0), turned to 180 degrees
Connections:
- net GND: no longer BATT.-
- net V_BATT: no longer BATT.+
Routing:
- net V_BATT: track 199.5 -> 270.7 mm, vias 5 -> 11
- net N$3: track 0.00 -> 33.7 mm
- net 5V: track 0.00 -> 25.7 mm
- net M_SWITCH: track 273.4 -> 287.8 mm
- net N$5: track 0.00 -> 4.35 mm
- net N$6: track 0.00 -> 3.13 mm
- net N$101: track 43.6 -> 42.2 mm
- net LSWITCH: track 507.7 -> 508.3 mm

Commit message: Hi
Other:
- outline, holes or cut-outs redrawn

Commit message: macOS
Parts:
- added ESC_IN: (no value), SparkFun-Connectors:1X03_LOCK
- added ESC_OUT: XT30PB-F, JH:XT30PB-F
- added Q37: AO3402, SparkFun-DiscreteSemi:SOT23-3
- added R8, R9: 4.7k, JH:R0603
- moved 1C6 23.1 mm to (-24.2, -79.2), turned to 270 degrees
- moved 1C10 13.1 mm to (-21.8, -71.7), turned to 90 degrees
- moved 1C7 9.83 mm to (-36.6, -68.4)
- moved 1C8 9.25 mm to (-28.8, -74.5)
- moved U2 9.17 mm to (-28.9, -78.6)
- moved 1R4 9.13 mm to (-31.3, -83.2)
- moved 1R3 9.04 mm to (-34.5, -80.5)
- moved 1D2 7.69 mm to (-21.8, -66.0), turned to 90 degrees
- moved 1C9 7.43 mm to (-37.8, -80.5), turned to 180 degrees
- moved S3 5.30 mm to (-21.1, -80.2)
- moved 1L2 3.36 mm to (-28.8, -68.5), turned to 270 degrees
Connections:
- new net 3.3V1: Q37.1, R9.1
- new net ESC_HV: ESC_IN.3, Q37.3, R8.2
- new net ESC_LV: Q37.2, R9.2
- new net GND1: ESC_IN.1
- new net N$7: ESC_IN.2
- net 5V: now also R8.1
- net GND: now also ESC_OUT.-
- net V_BATT: now also ESC_OUT.+
Routing:
- net V_BATT: track 270.7 -> 292.6 mm, vias 11 -> 9
- net GND: track 494.7 -> 508.5 mm, vias 63 -> 65
- net N$3: track 33.7 -> 24.7 mm
- net ESC_HV: track 0.00 -> 7.17 mm
- net 5V: track 25.7 -> 20.1 mm
- net BR_OUTA: track 34.7 -> 31.6 mm
- net GND_M: track 150.3 -> 152.9 mm, vias 13 -> 12
- net FR_OUTA: track 30.1 -> 28.1 mm
- net FR_PWM: track 135.1 -> 133.4 mm
- net FL_OUTB: track 34.6 -> 32.9 mm
- net FL_OUTA: track 32.7 -> 31.1 mm
- net 3.3V1: track 0.00 -> 1.48 mm
- net N$101: track 42.2 -> 43.6 mm
- net ESC_LV: track 0.00 -> 1.40 mm
- net VCCA: track 499.2 -> 500.5 mm
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- added copper zone on layer 1, net FR_OUTB
- removed copper zone on layer 1, net RFR_OUTB
Other:
- outline, holes or cut-outs redrawn
