File: Eagle PCB/Layer 3.brd (EAGLE design)
At the start: 108.5 x 108.5 mm, 78 parts, among them X1 SM06B-SRSS-TB, Y1 8MHz

Commit message: Done
Routing:
- net IR16: track 96.6 -> 98.1 mm
- net IR4: track 57.8 -> 56.5 mm
