File: Eagle PCB/Layer 3.brd (EAGLE design)
At the start: 108.5 x 108.5 mm, 88 parts, among them Q1 AO3402, Q2 AO3402, X1 SM06B-SRSS-TB, Y1 8MHz

Commit message: Hello
Parts:
- removed 3RD_LAYER: (no value), SparkFun-Connectors:1X05_LOCK
- removed ESC_IN, SERVO_IO: (no value), SparkFun-Connectors:1X03_LOCK
- removed ESC_OUT: XT30PB-F, JH:XT30PB-F
- removed Q1, Q2: AO3402, SparkFun-DiscreteSemi:SOT23-3
- removed R10, R11, R12, R13: 4.7k, JH:R0603
- moved U$14 2.49 mm to (15.8, 3.72), flipped to the bottom, turned to 180 degrees
Connections:
- removed net ESC_HV: ESC_IN.3, Q1.3, R10.2
- removed net N$4: ESC_IN.2
- removed net SERVO_HV: Q2.3, R12.2, SERVO_IO.3
- removed net V_BATT: ESC_OUT.+
- net 3.3V: no longer 3RD_LAYER.2, Q1.1, Q2.1, R11.1, R13.1
- net 5V: no longer 3RD_LAYER.5, R10.1, R12.1, SERVO_IO.2
- net ESC_LV: no longer 3RD_LAYER.4, Q1.2, R11.2
- net GND: no longer 3RD_LAYER.1, ESC_IN.1, ESC_OUT.-, SERVO_IO.1
- net SERVO_LV: no longer 3RD_LAYER.3, Q2.2, R13.2
Routing:
- net TX3_ST1: track 43.2 -> 36.1 mm
- net 3V3_SWITCH: track 509.5 -> 514.5 mm, vias 14 -> 16
- net BL_PWM: track 8.24 -> 12.8 mm
- net 3.3V: track 120.7 -> 116.5 mm
- net FL_PWM: track 8.28 -> 12.3 mm
- net FR_PWM: track 8.13 -> 12.0 mm
- net RX3_ST1: track 61.2 -> 65.0 mm
- net BATT_LVL: track 59.2 -> 62.5 mm
- net BR_PWM: track 9.29 -> 11.9 mm, vias 1 -> 2
- net LIGHT_INT: track 25.0 -> 27.4 mm
- net SWCLK: track 18.2 -> 16.0 mm
- net BL_DIR: track 38.9 -> 41.0 mm
- net FR_DIR: track 22.1 -> 20.1 mm
- net IR20: track 81.2 -> 79.4 mm
- net BR_DIR: track 37.0 -> 38.5 mm, vias 4 -> 5
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
Commit message: FUCK YOU
Parts:
- added 3RD_LAYER: (no value), SparkFun-Connectors:1X05_LOCK
- added ESC_IN, SERVO_IO: (no value), SparkFun-Connectors:1X03_LOCK
- added ESC_OUT: XT30PB-F, JH:XT30PB-F
- added Q1, Q2: AO3402, SparkFun-DiscreteSemi:SOT23-3
- added R10, R11, R12, R13: 4.7k, JH:R0603
Connections:
- new net ESC_HV: ESC_IN.3, Q1.3, R10.2
- new net N$4: ESC_IN.2
- new net SERVO_HV: Q2.3, R12.2, SERVO_IO.3
- new net V_BATT: ESC_OUT.+
- net 3.3V: now also 3RD_LAYER.2, Q1.1, Q2.1, R11.1, R13.1
- net 5V: now also 3RD_LAYER.5, R10.1, R12.1, SERVO_IO.2
- net ESC_LV: now also 3RD_LAYER.4, Q1.2, R11.2
- net GND: now also 3RD_LAYER.1, ESC_IN.1, ESC_OUT.-, SERVO_IO.1
- net SERVO_LV: now also 3RD_LAYER.3, Q2.2, R13.2

Commit message: Hi
Parts:
- moved BLUETOOTH 32.0 mm to (-1.54, -24.4)
Routing:
- net RX_BT: track 75.6 -> 33.9 mm, vias 8 -> 2
- net TX_BT: track 63.8 -> 36.0 mm, vias 6 -> 3
- net 3.3V: track 116.5 -> 121.4 mm, vias 5 -> 6
